File: V2/HW/HW.kicad_pcb (KiCad board)
At the start: 2 copper layers, 64 parts, among them J1 Power, J2 Conn_01x03, J3 Conn_01x13, J4 Conn_01x06, SW1 SW_Push, SW2 SW_Push, SW3 SW_Push, SW4 SW_Push, SW5 SW_Push, SW6 SW_Push, SW7 SW_Push, U1 74HC02, U10 W25Q32FVSS, U11 74AHC573, U12 SN74LV1T34DCK, U13 AS7C256, U14 74AHC573, U2 MCP1319MT-29LE-OT, U3 74HC08, U4 W25Q32FVSS, U5 AMS1117-3.3, U6 Caravel, U7 DAC7611, U8 SN74LV1T34DCK, U9 SN74LVC8T245, X1 15MHz

Commit message: V2 bring-up complete
Parts:
- added G***: LOGO, TholinsStuff:AvalonSemiLogo, F.Cu at (253.2, 129.2)
- U7: footprint Package_SO:SOIC-8_3.9x4.9mm_P1.27mm -> Package_DIP:DIP-8_W7.62mm
- moved SW4 146.6 mm to (250.2, 117.9)
- moved R5 143.2 mm to (256.3, 111.6)
- moved SW5 136.5 mm to (239.6, 127.0)
- moved SW3 136.2 mm to (239.3, 109.8)
- moved R7 135.5 mm to (252.2, 103.5)
- moved R9 134.0 mm to (246.1, 117.6), turned to 180 degrees
- moved R10 131.2 mm to (241.3, 124.1)
- moved D1 130.2 mm to (256.3, 109.1)
- moved R14 130.0 mm to (250.4, 111.5)
- moved R8 125.6 mm to (240.4, 106.6)
- moved R15 124.2 mm to (251.1, 89.5), turned to 180 degrees
- moved R17 122.0 mm to (251.1, 86.6), turned to 180 degrees
- moved SW6 121.8 mm to (228.4, 117.8)
- moved J3 121.7 mm to (217.6, 61.2)
- moved R20 121.4 mm to (252.5, 61.8)
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Routing:
- net GND: track 0.00 -> 133.8 mm, vias 0 -> 28
- net ADB6: track 0.00 -> 84.8 mm, vias 0 -> 4
- net PA4_TO1: track 0.00 -> 78.1 mm, vias 0 -> 4
- net 3V3_SDO: track 0.00 -> 70.8 mm, vias 0 -> 1
- net 3V3_SCLK: track 0.00 -> 66.7 mm, vias 0 -> 2
- net XCLK: track 0.00 -> 64.5 mm, vias 0 -> 2
- net PA5_PWM0: track 0.00 -> 61.3 mm, vias 0 -> 3
- net ~{POR}: track 0.00 -> 59.4 mm, vias 0 -> 2
- net ADB5: track 0.00 -> 57.8 mm, vias 0 -> 2
- net LE_LO: track 0.00 -> 53.3 mm, vias 0 -> 7
- net PB1_PWM2: track 0.00 -> 51.5 mm, vias 0 -> 1
- net Net-(U6-mprj_io[4]_SCK): track 0.00 -> 50.7 mm, vias 0 -> 1
- net IOC: track 0.00 -> 50.5 mm, vias 0 -> 3
- net ADB2: track 0.00 -> 50.3 mm, vias 0 -> 3
- net ADB4: track 0.00 -> 49.6 mm, vias 0 -> 2
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- added copper zone on B.Cu, net +3V3
- added copper zone on F.Cu, net +5V
- added copper zone on In1.Cu, net +5V
- added copper zone on In2.Cu, net GND
Other:
- board outline added: 54.9 x 75.8 mm
- copper layers 2 -> 4
- board text added: "+5V"
- board text added: "AS2650-2 bring-up 2024-08-29 0094"
- board text added: "CC0 / C"
- board text added: "CC1 / IDC"
- board text added: "Caravel OK"
- board text added: "GND"
