File: V2/HW/HW.kicad_sch (KiCad schematic)
At the start: 64 parts, among them J1 Power, J2 Conn_01x03, J3 Conn_01x13, J4 Conn_01x06, SW1 SW_Push, SW2 SW_Push, SW3 SW_Push, SW4 SW_Push, SW5 SW_Push, SW6 SW_Push, SW7 SW_Push, U1 74HC02, U10 W25Q32FVSS, U11 74AHC573, U12 SN74LV1T34DCK, U13 AS7C256, U14 74AHC573, U2 MCP1319MT-29LE-OT, U3 74HC08, U4 W25Q32FVSS, U5 AMS1117-3.3, U6 Caravel, U7 DAC7611, U8 SN74LV1T34DCK, U9 SN74LVC8T245, X1 15MHz

Commit message: V2 bring-up complete
Parts:
- U7: footprint Package_SO:SOIC-8_3.9x4.9mm_P1.27mm -> Package_DIP:DIP-8_W7.62mm
Changed lines of the file:
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@@
 			)
 		)
-		(property "Footprint" "Package_SO:SOIC-8_3.9x4.9mm_P1.27mm"
+		(property "Footprint" "Package_DIP:DIP-8_W7.62mm"
 			(at 119.38 124.46 0)
 			(effects
