File: V2/MinimalSetup/KiCad/MinimalSetup.kicad_sch (KiCad schematic)
At the start: 9 parts, among them U1 gfmpw-breakout, U2 W25Q32, Y1 max. 50MHz

Commit message: MinimalExample fixes
Parts:
- Y1: value max. 50MHz -> 15MHz
Changed lines of the file:
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@@
 			)
 		)
-		(property "Value" "max. 50MHz"
+		(property "Value" "15MHz"
 			(at 102.87 26.5998 0)
 			(effects
